Commit message: cartograper3d

File: vlp16-imu.urdf (robot description, URDF)
Before this commit: robot stencil, 3 links, 2 joints
Links:
- removed link map
- added link imu_link; visual box size=0.06 0.04 0.02
Joints:
- removed joint map_joint
- added joint imu_link_joint: type fixed, parent base_link, child imu_link, origin xyz=0 0 0 rpy=0 0 0
